File: schematic/bldcshieldbackup.brd (EAGLE design)
At the start: 51 parts, among them IC3 IR2101SMD, IC4 IR2101SMD, IC5 IR2101SMD

Commit message: redoing brf layout from scatch
deleted gerbers and backed up brd file
Routing:
- net S$1: track 252.3 -> 0.00 mm
Other:
- board text added: "Open BLDC 0.1"
- board text added: "www.OpenRover.com"
