File: schematic/bldcshield.brd (EAGLE design)
At the start: 97 x 53.3 mm, 43 parts, among them IC1 IR2101SMD, IC2 IR2101SMD, IC3 IR2101SMD, Q1 BUZ11BV, Q2 BUZ11BV, Q3 BUZ11BV, Q4 BUZ11BV, Q5 BUZ11BV, Q6 BUZ11BV, Q8 Shield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

Commit message: working on new layout and swapped all transistors and wire pads.  Need to look at better IO assignment and redo power supply.
Parts:
- removed +: Vcc, wirepad:3,81/1,4
- removed -: (no value), wirepad:3,81/1,4
- removed IC1, IC2, IC3: IR2101SMD, IR:SO08
- added GND, VCC: (no value), wirepad:4,16O1,6
- added U2, U3, U4: IR2101SOIC-8, SnapEDA-Library:SOIC127P490X600X175-8N
- BLDC1, BLDC2, BLDC3: device wirepad:3,81/1,4 -> wirepad:4,16O1,6
- Q8: device adafruit:ARDUINOR3-BLDC -> adafruit:ARDUINOR3-NOTEXT-NOIOREF
- U1: value V_REG_317SINK -> LM5007; device SparkFun-PowerIC:TO220-ADJ -> SparkFun-PowerIC:MSOP-8-EP
- moved U1 51.9 mm to (18.0, 9.91), turned to 0 degrees
- moved Q1 12.6 mm to (38.6, 35.1), turned to 180 degrees
- moved Q4 12.4 mm to (50.0, 35.1), turned to 180 degrees
- moved Q6 12.3 mm to (73.2, 35.3), turned to 180 degrees
- moved Q3 12.2 mm to (61.5, 35.1), turned to 180 degrees
- moved Q5 12.1 mm to (84.6, 35.3), turned to 180 degrees
- moved Q2 11.9 mm to (27.2, 35.1), turned to 180 degrees
- moved R28 2.81 mm to (92.7, 48.8)
- moved C8 2.81 mm to (92.2, 57.9)
- moved R27 2.81 mm to (92.3, 53.0)
- moved BLDC3 2.05 mm to (78.7, 43.9)
- moved BLDC2 1.80 mm to (55.6, 43.7)
- moved BLDC1 1.80 mm to (32.8, 43.7)
Connections:
- removed net N$17: C5.2, D3.C, IC3.8
- removed net N$25: C4.2, D2.C, IC2.8
- removed net N$33: C1.2, D1.C, IC1.8
- new net VB: C1.2, C4.2, C5.2, D1.C, D2.C, D3.C, U2.8, U3.8, U4.8
- net +12V: now also U2.1, U3.1, U4.1; no longer IC1.1, IC2.1, IC3.1, U1.OUT
- net BLDC1: now also U2.6; no longer IC1.6
- net BLDC2: now also U3.6; no longer IC2.6
- net BLDC3: now also U4.6; no longer IC3.6
- net GND: now also GND.1, U2.4, U3.4, U4.4; no longer -.1, IC1.4, IC2.4, IC3.4
- net HI_2: now also U3.2; no longer IC2.2
- net HI_3: now also U4.2; no longer IC3.2
- net LO_2: now also U3.3; no longer IC2.3
- net LO_3: now also U4.3; no longer IC3.3
- net N$13: now also U4.7; no longer IC3.7
- net N$16: now also U4.5; no longer IC3.5
- net N$2: no longer U1.ADJ
- net N$21: now also U3.7; no longer IC2.7
- net N$24: now also U3.5; no longer IC2.5
- net N$29: no longer IC1.7
- net N$32: no longer IC1.5
- net N$4: now also U2.2; no longer IC1.2
- net N$8: now also U2.3; no longer IC1.3
- net VCC: now also VCC.1; no longer +.1, U1.IN
Routing:
- net VB: track 0.00 -> 50.4 mm
- net N$17: track 16.7 -> 0.00 mm
- net N$25: track 16.4 -> 0.00 mm
- net N$33: track 16.1 -> 0.00 mm
- net N$14: track 18.3 -> 33.9 mm
- net N$30: track 31.5 -> 17.3 mm, vias 1 -> 0
- net N$15: track 34.4 -> 24.4 mm
- net VCC: track 25.1 -> 15.7 mm
- net N$16: track 7.52 -> 0.08 mm
- net N$31: track 18.1 -> 25.2 mm, vias 0 -> 2
- net N$23: track 24.4 -> 17.3 mm, vias 2 -> 0
- net N$1: track 26.1 -> 20.3 mm, vias 2 -> 0
- net CURRENT: track 23.2 -> 17.9 mm
- net BLDC1: track 40.1 -> 37.7 mm
- net BLDC3: track 40.7 -> 38.4 mm
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
Commit message: added pdfs for new parts
Connections:
- removed net N$29: R3.2
- removed net N$32: R6.2
- removed net VB: C1.2, C4.2, C5.2, D1.C, D2.C, D3.C, U2.8, U3.8, U4.8
- new net N$10: R6.2, U2.5
- new net N$11: R3.2, U2.7
- new net VB1: C1.2, D1.C, U2.8
- new net VB2: C4.2, D2.C, U3.8
- new net VB3: C5.2, D3.C, U4.8
- net HI_2: now also Q8.D10; no longer Q8.D9
- net HI_3: now also Q8.D9; no longer Q8.D5
- net LO_2: now also Q8.D6; no longer Q8.D8
- net LO_3: now also Q8.D5; no longer Q8.D13
- net N$4: now also Q8.D11; no longer Q8.D4
- net N$5: now also Q8.D4, R7.1; no longer Q8.D1, R5.1
- net N$6: now also Q8.D3, R5.1; no longer Q8.D2, R7.1
- net N$7: now also Q8.D2; no longer Q8.D0
- net N$8: now also Q8.D7; no longer Q8.D12
Routing:
- net VB: track 50.4 -> 0.00 mm
- net N$4: track 52.5 -> 20.0 mm, vias 1 -> 0
- net VB1: track 0.00 -> 16.9 mm
- net VB2: track 0.00 -> 16.8 mm
- net VB3: track 0.00 -> 16.7 mm
- net LO_3: track 21.3 -> 11.1 mm
- net N$8: track 23.9 -> 33.6 mm, vias 0 -> 1
- net N$11: track 0.00 -> 8.83 mm
- net N$10: track 0.00 -> 8.29 mm
- net N$29: track 8.07 -> 0.00 mm
- net N$24: track 8.01 -> 0.32 mm
- net N$32: track 7.46 -> 0.00 mm
- net N$16: track 0.08 -> 7.53 mm
- net LO_2: track 13.6 -> 20.8 mm
- net HI_3: track 8.81 -> 13.4 mm
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
Commit message: generated gerbers for new boards.  might need some small tweaks on the keep out zones.
Parts:
- added C10, C11, C7: 100nF, SmartPrj:C1206
- added C12: 33uF, SparkFun-Capacitors:PANASONIC_C
- added C6: 22uF, SparkFun-Capacitors:PANASONIC_C
- added C9: 10nF, SmartPrj:C1206
- added D4: BAS70-05DPAK, SCHOTTKY:DPAK229P990X238-3N
- added D5: (no value), smf_11:SOD123F
- added D6: (no value), diode:SOD123
- added L1: 100uH, SparkFun-Passives:INDUCTOR-SRP4020
- added R8: 1k, SmartPrj:R1206
- added R9: 3.01k, SmartPrj:R1206
- C24: value 1uF -> 100nF
- C25: value 0.1u -> 100nF
- R32: value 240 -> 100k
- R33: value 2.2k -> 200k
- moved U1 105.7 mm to (104.9, 70.1), turned to 270 degrees
- moved R33 84.6 mm to (112.3, 68.6)
- moved C25 76.2 mm to (101.9, 55.4)
- moved R32 71.9 mm to (99.1, 66.8)
- moved C24 51.7 mm to (85.3, 62.0), turned to 90 degrees
Connections:
- new net N$12: R33.1, U1.6
- new net N$17: C9.2, U1.2
- new net N$18: C7.2, U1.7
- new net N$19: C9.1, D6.C, L1.P$1, U1.1
- new net N$20: R32.1, U1.3
- new net N$26: R8.1, R9.2, U1.5
- net +12V: now also C10.2, C11.2, C12.+, L1.P$2, R9.1; no longer R32.1
- net GND: now also C10.1, C11.1, C12.-, C6.-, C7.1, D5.A, D6.A, R32.2, R8.2, U1.4, U1.EP; no longer R33.2
- net N$2: now also C25.2, C6.+, D4.4, D5.C, R33.2, U1.8; no longer R32.2, R33.1
- net VCC: now also D4.1, D4.3; no longer C25.2
Routing:
- net N$2: track 7.00 -> 40.2 mm
- net +12V: track 78.2 -> 105.6 mm
- net VCC: track 15.7 -> 43.1 mm
- net N$19: track 0.00 -> 16.9 mm
- net N$17: track 0.00 -> 9.34 mm
- net N$26: track 0.00 -> 8.09 mm
- net N$24: track 0.32 -> 8.01 mm
- net N$20: track 0.00 -> 4.83 mm
- net N$12: track 0.00 -> 4.04 mm
- net N$18: track 0.00 -> 2.76 mm
- net GND: vias 1 -> 4
