File: schematic2/two_pieceboard_1.brd (EAGLE design)
At the start: 81.3 x 53.3 mm, 39 parts, among them IC1 IR2101SMD, IC2 IR2101SMD, IC3 IR2101SMD, Q1 MOSFET-NCHANNELFDD8580, Q2 MOSFET-NCHANNELFDD8580, Q3 Shield, Q4 MOSFET-NCHANNELFDD8580, Q5 MOSFET-NCHANNELFDD8580, Q6 MOSFET-NCHANNELFDD8580, Q7 MOSFET-NCHANNELFDD8580, U3 LM317DCY

Commit message: started working on board one
Parts:
- removed C24: 1uF, SmartPrj:C1206
- removed C25: 0.1u, SmartPrj:C1206
- removed Q1, Q2, Q4, Q5, Q6, Q7: MOSFET-NCHANNELFDD8580, SparkFun:DPAK
- removed Q3: Shield, adafruit:ARDUINOR3-BLDC
- removed R27: 4.7k, SmartPrj:R1206
- removed R28: 0.001, resistor:R2512
- removed R32: 240, SmartPrj:R1206
- removed R33: 2.2k, SmartPrj:R1206
- removed U3: LM317DCY, Texas Instruments_By_element14_Batch_1:SOT230P700X180-4N
- removed X1: (no value), con-phoenix-508:MKDSN1,5/2-5,08
- removed X2: (no value), con-phoenix-508:MKDSN1,5/3-5,08
- added C3, C6, C7: 100nf, SmartPrj:C1206
- added D4, D5, D6: MMSD914, diode:SOD123
- added IC4, IC5, IC6: IR2101SMD, IR:SO08
- added JP2: (no value), SparkFun-Connectors:2X03
- added R10, R12, R13, R15, R8, R9: 22, SmartPrj:R1206
- added R16, R17, R18: 10k, SmartPrj:R1206
- added R20: 200K, SmartPrj:R1206
- added R21: 68k, SmartPrj:R1206
- added SV1: (no value), con-lsta:FE08-2
- added SV2: (no value), con-lsta:FE10-2
- added SV3: (no value), con-lsta:FE15-2
- added SV4: (no value), con-lsta:FE17-2
- moved C8 167.5 mm to (19.1, -94.7), flipped to the top, turned to 0 degrees
Connections:
- removed net +3V3: Q3.3V
- removed net BLDC1: C1.1, IC1.6, Q1.3, Q2.4, X2.1
- removed net CURRENT: Q2.3, Q3.A4, Q5.3, Q7.3, R27.2, R28.2
- removed net HI_1: IC1.2, Q3.D13
- removed net HI_2: IC2.2, Q3.D11
- removed net HI_3: IC3.2, Q3.D9
- removed net LOW_VOLTAGE: C2.2, Q3.A3, R1.1, R2.2
- removed net LO_1: IC1.3, Q3.D12
- removed net LO_2: IC2.3, Q3.D10
- removed net LO_3: IC3.3, Q3.D8
- removed net VCC: C25.2, Q1.4, Q4.4, Q6.4, R1.2, U3.3, X1.1
- new net BLDC4: C6.1, IC5.6
- new net BLDC5: C3.1, IC4.6
- new net HI_1_A: IC1.2
- new net HI_1_B: IC6.2
- new net HI_2_A: IC2.2
- new net HI_2_B: IC5.2
- new net HI_3_A: IC3.2
- new net HI_3_B: IC4.2
- new net LOW_VOLTAGE1: C2.2, R1.1, R2.2
- new net LOW_VOLTAGE2: C8.2, R20.1, R21.2
- new net LO_1_A: IC1.3
- new net LO_1_B: IC6.3
- new net LO_2_A: IC2.3
- new net LO_2_B: IC5.3
- new net LO_3_A: IC3.3
- new net LO_3_B: IC4.3
- new net N$11: R8.1
- new net N$12: IC4.5, R8.2
- new net N$18: C3.2, D4.C, IC4.8
- new net N$19: IC5.7, R12.2
- new net N$20: R10.1
- new net N$22: IC5.5, R10.2
- new net N$26: C6.2, D5.C, IC5.8
- new net N$27: IC6.7, R15.2
- new net N$28: R13.1
- new net N$34: C7.2, D6.C, IC6.8
- new net N$35: R12.1
- new net N$37: C7.1, IC6.6
- new net N$38: R15.1
- new net N$39: JP2.6, R16.1
- new net N$40: JP2.4, R17.1
- new net N$41: JP2.2, R18.1
- new net N$6: R3.1
- new net N$8: IC4.7, R9.2
- net +12V: now also D4.A, D5.A, D6.A, IC4.1, IC5.1, IC6.1, R1.2, R20.2; no longer C24.2, R32.1, U3.2, U3.4
- net +5V: now also JP2.1, R16.2, R17.2, R18.2; no longer Q3.5V, Q3.VIN
- net BLDC2: no longer Q4.3, Q5.4, X2.2
- net BLDC3: no longer Q6.3, Q7.4, X2.3
- net GND: now also IC4.4, IC5.4, IC6.4, JP2.5, R21.1; no longer C24.1, C25.1, Q3.GND, Q3.GND1, Q3.GND2, R28.1, R33.2, X1.2
- net N$1: no longer Q4.1
- net N$10: no longer Q3.A1
- net N$14: no longer Q6.1
- net N$15: no longer Q7.1
- net N$23: no longer Q5.1
- net N$30: now also IC6.5, R13.2; no longer Q1.1, R3.1
- net N$31: no longer Q2.1
- net N$4: no longer Q3.A2
- net N$5: now also C1.1, IC1.6; no longer R32.2, R33.1, U3.1
- net N$7: no longer Q3.A0
- net N$9: now also R9.1; no longer C8.2, R27.1
Routing:
- net VCC: track 118.9 -> 0.00 mm, vias 2 -> 0
- net +12V: track 85.6 -> 179.4 mm, vias 0 -> 2
- net LO_3: track 67.4 -> 0.00 mm, vias 1 -> 0
- net LO_3_A: track 0.00 -> 66.9 mm, vias 0 -> 1
- net HI_3: track 63.7 -> 0.00 mm, vias 1 -> 0
- net HI_3_A: track 0.00 -> 63.5 mm, vias 0 -> 1
- net LO_2: track 50.4 -> 0.00 mm, vias 1 -> 0
- net LO_2_A: track 0.00 -> 49.9 mm, vias 0 -> 1
- net HI_2: track 48.1 -> 0.00 mm, vias 1 -> 0
- net HI_2_A: track 0.00 -> 47.9 mm, vias 0 -> 1
- net BLDC1: track 38.6 -> 0.00 mm
- net LO_1: track 34.3 -> 0.00 mm, vias 1 -> 0
- net LO_1_A: track 0.00 -> 34.0 mm, vias 0 -> 1
- net HI_1: track 31.1 -> 0.00 mm, vias 1 -> 0
- net HI_1_A: track 0.00 -> 30.3 mm, vias 0 -> 1
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- added copper zone on layer 16, net CURRENT2
- removed copper zone on layer 16, net CURRENT

Commit message: stated working on main shield  got connectors to FET boards done.
Parts:
- added J1, J2: 2X6 FEMALE, SparkFun-Connectors:2X6
Connections:
- removed net +12V: D1.A, D2.A, D3.A, D4.A, D5.A, D6.A, IC1.1, IC2.1, IC3.1, IC4.1, IC5.1, IC6.1, R1.2, R20.2
- removed net BLDC2: C4.1, IC2.6
- removed net BLDC3: C5.1, IC3.6
- removed net BLDC4: C6.1, IC5.6
- removed net BLDC5: C3.1, IC4.6
- removed net N$1: R11.1
- removed net N$11: R8.1
- removed net N$14: R19.1
- removed net N$15: R22.1
- removed net N$20: R10.1
- removed net N$23: R14.1
- removed net N$28: R13.1
- removed net N$31: R6.1
- removed net N$35: R12.1
- removed net N$37: C7.1, IC6.6
- removed net N$38: R15.1
- removed net N$5: C1.1, IC1.6
- removed net N$6: R3.1
- removed net N$9: R9.1
- new net +12V_A: D1.A, D2.A, D3.A, IC1.1, IC2.1, IC3.1, J1.1, R1.2
- new net +12V_B: D4.A, D5.A, D6.A, IC4.1, IC5.1, IC6.1, J2.1, R20.2
- new net BLDC1_A: C1.1, IC1.6, J1.4
- new net BLDC1_B: C7.1, IC6.6, J2.4
- new net BLDC2_A: C4.1, IC2.6, J1.11
- new net BLDC2_B: C6.1, IC5.6, J2.11
- new net BLDC3_A: C5.1, IC3.6, J1.9
- new net BLDC3_B: C3.1, IC4.6, J2.9
- new net CURRENT_A: J1.3
- new net CURRENT_B: J2.3
- new net GATE_HI_1_A: J1.12, R3.1
- new net GATE_HI_1_B: J2.12, R15.1
- new net GATE_HI_2_A: J1.5, R11.1
- new net GATE_HI_2_B: J2.5, R12.1
- new net GATE_HI_3_A: J1.7, R19.1
- new net GATE_HI_3_B: J2.7, R9.1
- new net GATE_LO_1_A: J1.10, R6.1
- new net GATE_LO_1_B: J2.10, R13.1
- new net GATE_LO_2_A: J1.8, R14.1
- new net GATE_LO_2_B: J2.8, R10.1
- new net GATE_LO_3_A: J1.6, R22.1
- new net GATE_LO_3_B: J2.6, R8.1
- net GND: now also J1.2, J2.2
Routing:
- net +12V_A: track 0.00 -> 179.4 mm, vias 0 -> 2
- net +12V: track 179.4 -> 0.00 mm, vias 2 -> 0
- net BLDC3_A: track 0.00 -> 58.3 mm, vias 0 -> 6
- net BLDC3: track 58.3 -> 0.00 mm, vias 6 -> 0
- net N$14: track 50.3 -> 0.00 mm, vias 2 -> 0
- net GATE_HI_3_A: track 0.00 -> 50.3 mm, vias 0 -> 2
- net BLDC2_A: track 0.00 -> 41.4 mm, vias 0 -> 6
- net BLDC2: track 41.4 -> 0.00 mm, vias 6 -> 0
- net N$15: track 32.5 -> 0.00 mm, vias 1 -> 0
- net GATE_LO_3_A: track 0.00 -> 32.5 mm, vias 0 -> 1
- net N$31: track 31.3 -> 0.00 mm, vias 3 -> 0
- net GATE_LO_1_A: track 0.00 -> 31.3 mm, vias 0 -> 3
- net N$1: track 27.1 -> 0.00 mm, vias 2 -> 0
- net GATE_HI_2_A: track 0.00 -> 27.1 mm, vias 0 -> 2
- net N$23: track 25.2 -> 0.00 mm, vias 3 -> 0
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- added copper zone on layer 1, net +12V_B
- added copper zone on layer 1, net BLDC2_A
- added copper zone on layer 16, net BLDC2_A
- added copper zone on layer 1, net BLDC3_A
- added copper zone on layer 16, net BLDC3_A
- removed copper zone on layer 1, net BLDC2
- removed copper zone on layer 16, net BLDC2
- removed copper zone on layer 1, net BLDC3
- removed copper zone on layer 16, net BLDC3
- removed copper zone on layer 1, net VCC
