File: schematic2/two_pieceboard_1.sch (EAGLE design)
At the start: 48 parts, among them IC1 IR2101SMD, IC2 IR2101SMD, IC3 IR2101SMD, IC4 IR2101SMD, IC5 IR2101SMD, IC6 IR2101SMD

Commit message: stated working on main shield  got connectors to FET boards done.
Parts:
- added J1, J2: 2X6 FEMALE, SparkFun-Connectors:M06X2PTH_FEMALE
Connections:
- removed net +12V: D1.A, D2.A, D3.A, D4.A, D5.A, D6.A, IC1.VCC, IC2.VCC, IC3.VCC, IC4.VCC, IC5.VCC, IC6.VCC, R1.2, R20.2
- removed net BLDC2: C4.1, IC2.VS
- removed net BLDC3: C5.1, IC3.VS
- removed net BLDC4: C6.1, IC5.VS
- removed net BLDC5: C3.1, IC4.VS
- removed net N$1: R11.1
- removed net N$11: R8.1
- removed net N$14: R19.1
- removed net N$15: R22.1
- removed net N$20: R10.1
- removed net N$23: R14.1
- removed net N$28: R13.1
- removed net N$31: R6.1
- removed net N$35: R12.1
- removed net N$37: C7.1, IC6.VS
- removed net N$38: R15.1
- removed net N$5: C1.1, IC1.VS
- removed net N$6: R3.1
- removed net N$9: R9.1
- new net +12V_A: D1.A, D2.A, D3.A, IC1.VCC, IC2.VCC, IC3.VCC, J1.1, R1.2
- new net +12V_B: D4.A, D5.A, D6.A, IC4.VCC, IC5.VCC, IC6.VCC, J2.1, R20.2
- new net BLDC1_A: C1.1, IC1.VS, J1.4
- new net BLDC1_B: C7.1, IC6.VS, J2.4
- new net BLDC2_A: C4.1, IC2.VS, J1.11
- new net BLDC2_B: C6.1, IC5.VS, J2.11
- new net BLDC3_A: C5.1, IC3.VS, J1.9
- new net BLDC3_B: C3.1, IC4.VS, J2.9
- new net CURRENT_A: J1.3
- new net CURRENT_B: J2.3
- new net GATE_HI_1_A: J1.12, R3.1
- new net GATE_HI_1_B: J2.12, R15.1
- new net GATE_HI_2_A: J1.5, R11.1
- new net GATE_HI_2_B: J2.5, R12.1
- new net GATE_HI_3_A: J1.7, R19.1
- new net GATE_HI_3_B: J2.7, R9.1
- new net GATE_LO_1_A: J1.10, R6.1
- new net GATE_LO_1_B: J2.10, R13.1
- new net GATE_LO_2_A: J1.8, R14.1
- new net GATE_LO_2_B: J2.8, R10.1
- new net GATE_LO_3_A: J1.6, R22.1
- new net GATE_LO_3_B: J2.6, R8.1
- net GND: now also J1.2, J2.2
