File: schematic/recon_switcher/bldcshield.brd (EAGLE design)
At the start: 97 x 53.3 mm, 55 parts, among them Q1 BUZ11BV, Q2 BUZ11BV, Q3 BUZ11BV, Q4 BUZ11BV, Q5 BUZ11BV, Q6 BUZ11BV, Q8 Shield, U1 LM5007, U2 IR2101SOIC-8, U3 IR2101SOIC-8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

Commit message: tweaked lm507 board and made copy and created a board based on recon switcher.
Parts:
- removed C12: 33uF, SparkFun-Capacitors:PANASONIC_C
- removed C24, C7: 100nF, SmartPrj:C1206
- removed C9: 10nF, SmartPrj:C1206
- removed D6: (no value), diode:SOD123
- removed L1: 100uH, SparkFun-Passives:INDUCTOR-SRP4020
- removed R32: 100k, SmartPrj:R1206
- removed R33: 200k, SmartPrj:R1206
- removed R8: 1k, SmartPrj:R1206
- removed R9: 3.01k, SmartPrj:R1206
- C6: value 22uF -> (none); device SparkFun-Capacitors:PANASONIC_C -> SparkFun-Capacitors:CPOL-RADIAL-100UF-25V
- U1: value LM5007 -> R-785.0-0.5; device SparkFun-PowerIC:MSOP-8-EP -> R-785.0-0.5:RECOM_R-785.0-0.5
- moved C6 22.1 mm to (95.2, 72.6), turned to 270 degrees
- moved U1 0.51 mm to (104.9, 70.6), turned to 180 degrees
Connections:
- removed net N$12: R33.1, U1.6
- removed net N$17: C9.2, U1.2
- removed net N$18: C7.2, U1.7
- removed net N$19: C9.1, D6.C, L1.P$1, U1.1
- removed net N$20: R32.1, U1.3
- removed net N$26: R8.1, R9.2, U1.5
- net +12V: now also C6.1, U1.3; no longer C12.+, C24.2, L1.P$2, R9.1
- net GND: now also C6.2, U1.2; no longer C12.-, C24.1, C6.-, C7.1, D6.A, R32.2, R8.2, U1.4, U1.EP
- net N$2: now also U1.1; no longer C6.+, R33.2, U1.8
Routing:
- net N$19: track 16.9 -> 0.00 mm
- net N$2: track 40.2 -> 28.2 mm
- net N$17: track 9.34 -> 0.00 mm
- net N$26: track 8.09 -> 0.00 mm
- net N$20: track 4.83 -> 0.00 mm
- net +12V: track 105.6 -> 101.5 mm
- net N$12: track 4.04 -> 0.00 mm
- net N$18: track 2.76 -> 0.00 mm
